Commit message: edit urdf

File: aba_excavator/excavator.urdf (robot description, URDF)
Before this commit: robot excavator, 8 links, 7 joints
Links:
- added link Link_EE, mass 0; visual sphere radius=0.1
Joints:
- added joint Joint_EE: type fixed, parent link5, child Link_EE, origin xyz=2 0 -0.75 rpy=0 0 0, axis 1 0 0

Commit message: trajectoriees

File: aba_excavator/excavator.urdf (robot description, URDF)
Before this commit: robot excavator, 9 links, 8 joints
Links:
- link Link_EE: geometry visual sphere radius=0.0001
